File: DMH_S_H_Noise_PCB_Conn/DMH_S_H_Noise_PCB_Conn.kicad_sch (KiCad schematic)
At the start: 0 parts

Commit message: Finished connectors PCB
Connections:
- no-connect marks 0 -> 11
Other:
- removed sheet Core Circuit
- removed sheet Power
- sheet Inputs and Outputs ports: added Blue, Clock Out, External Clock, Input, Internal Clock, Pink, S&H, S&H Out, Slew In, Slew Out, White; removed none
Changed lines of the file:
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@@
 		(comment 1 "PCB for 5 cm Kosmo format synthesizer module")
 	)
-	(sheet
-		(at 260.35 16.51)
-		(size 20.32 27.94)
-		(fields_autoplaced yes)
-		(stroke
-			(width 0.1524)
-			(type solid)
-		)
-		(fill
-			(color 0 0 0 0.0000)
-		)
-		(property "Sheetname" "Power"
-			(at 260.35 15.7984 0)
-			(effects
-				(font
-					(size 1.27 1.27)
-				)
-				(justify left bottom)
-			)
-		)
-		(property "Sheetfile" "Power.kicad_sch"
-			(at 260.35 45.0346 0)
-			(effects
-				(font
-					(size 1.27 1.27)
-				)
-				(justify left top)
-				(hide yes)
-			)
-		)
-		(pin "Bus Gate" output
-			(at 260.35 25.4 180)
-			(effects
-				(font
-					(size 1.27 1.27)
-				)
-				(justify left)
-			)
-		)
-		(pin "Bus CV" output
-			(at 260.35 34.29 180)
-			(effects
-				(font
-					(size 1.27 1.27)
-				)
-				(justify left)
-			)
-		)
-		(instances
-			(project "DMH-Kosmo-5cm-PCB"
-				(path "/58f4306d-5387-4983-bb08-41a2313fd315"
-					(page "4")
-				)
-			)
-		)
+	(no_connect
+		(at 38.1 72.39)
+	)
+	(no_connect
+		(at 38.1 106.68)
+	)
+	(no_connect
+		(at 38.1 76.2)
+	)
+	(no_connect
+		(at 38.1 80.01)
+	)
+	(no_connect
+		(at 38.1 95.25)
+	)
+	(no_connect
+		(at 38.1 83.82)
+	)
+	(no_connect
+		(at 38.1 99.06)
+	)
+	(no_connect
+		(at 38.1 87.63)
+	)
+	(no_connect
+		(at 38.1 68.58)
+	)
+	(no_connect
+		(at 38.1 102.87)
+	)
+	(no_connect
+		(at 38.1 91.44)
 	)
 	(sheet
-		(at 120.65 80.01)
-		(size 41.91 38.1)
-		(fields_autoplaced yes)
-		(stroke
-			(width 0.1524)
-			(type solid)
-		)
-		(fill
-			(color 0 0 0 0.0000)
-		)
-		(property "Sheetname" "Core Circuit"
-			(at 120.65 79.2984 0)
-			(effects
-				(font
-					(size 1.27 1.27)
-				)
-				(justify left bottom)
-			)
-		)
-		(property "Sheetfile" "Core_Circuit.kicad_sch"
-			(at 120.65 118.6946 0)
-			(effects
-				(font
-					(size 1.27 1.27)
-				)
-				(justify left top)
-				(hide yes)
-			)
-		)
-		(instances
-			(project "DMH-Kosmo-5cm-PCB"
-				(path "/58f4306d-5387-4983-bb08-41a2313fd315"
-					(page "3")
-				)
-			)
-		)
-	)
-	(sheet
-		(at 17.78 17.78)
-		(size 20.32 118.11)
+		(at 17.78 63.5)
+		(size 20.32 50.8)
 		(fields_autoplaced yes)
 		(stroke
@@
 		)
 		(property "Sheetname" "Inputs and Outputs"
-			(at 17.78 17.0684 0)
+			(at 17.78 62.7884 0)
 			(effects
 				(font
@@
 		)
 		(property "Sheetfile" "Inputs_and_Outputs.kicad_sch"
-			(at 17.78 136.4746 0)
+			(at 17.78 114.8846 0)
 			(effects
 				(font
@@
 			)
 		)
+		(pin "S&H" input
+			(at 38.1 80.01 0)
+			(effects
+				(font
+					(size 1.27 1.27)
+				)
+				(justify right)
+			)
+		)
+		(pin "Internal Clock" input
+			(at 38.1 72.39 0)
+			(effects
+				(font
+					(size 1.27 1.27)
+				)
+				(justify right)
+			)
+		)
+		(pin "External Clock" output
+			(at 38.1 76.2 0)
+			(effects
+				(font
+					(size 1.27 1.27)
+				)
+				(justify right)
+			)
+		)
+		(pin "Clock Out" input
+			(at 38.1 68.58 0)
+			(effects
+				(font
+					(size 1.27 1.27)
+				)
+				(justify right)
+			)
+		)
+		(pin "Slew In" output
+			(at 38.1 83.82 0)
+			(effects
+				(font
+					(size 1.27 1.27)
+				)
+				(justify right)
+			)
+		)
+		(pin "Input" output
+			(at 38.1 87.63 0)
+			(effects
+				(font
+					(size 1.27 1.27)
+				)
+				(justify right)
+			)
+		)
+		(pin "White" input
+			(at 38.1 102.87 0)
+			(effects
+				(font
+					(size 1.27 1.27)
+				)
+				(justify right)
+			)
+		)
+		(pin "Slew Out" input
+			(at 38.1 95.25 0)
+			(effects
+				(font
+					(size 1.27 1.27)
+				)
+				(justify right)
+			)
+		)
+		(pin "Pink" input
+			(at 38.1 106.68 0)
+			(effects
+				(font
+					(size 1.27 1.27)
+				)
+				(justify right)
+			)
+		)
+		(pin "Blue" input
+			(at 38.1 99.06 0)
+			(effects
+				(font
+					(size 1.27 1.27)
+				)
+				(justify right)
+			)
+		)
+		(pin "S&H Out" input
+			(at 38.1 91.44 0)
+			(effects
+				(font
+					(size 1.27 1.27)
+				)
+				(justify right)
+			)
+		)
 		(instances
-			(project "DMH-Kosmo-5cm-PCB"
+			(project "DMH_S_H_Noise_PCB_Conn"
 				(path "/58f4306d-5387-4983-bb08-41a2313fd315"
 					(page "2")
