File: DMH_S_H_Noise_PCB_Conn/Inputs_and_Outputs.kicad_sch (KiCad schematic)
At the start: 0 parts

Commit message: Finished connectors PCB
Parts:
- added J1, J2, J3, J4, J5, J6, J7, J8, J9: TS_Jack_6.35mm_Sw, SynthStuff:CUI_MJ-63052A, symbol SynthStuff:TS_Jack_6.35mm_Sw
- added J200: IDC_02x05, SynthStuff:IDC-Header_2x05_P2.54mm_Vertical_BackBone, symbol SynthStuff:BackBone_Connector_10Pin
- added J50, J60, J70: Conn_01x06, Connector_PinHeader_2.54mm:PinHeader_1x06_P2.54mm_Vertical, symbol Connector_Generic:Conn_01x06
Connections:
- new net: J200.1 (Pin_1), J4.TN, J70.1 (Pin_1)
- new net: J200.2 (Pin_2), J5.TN, J70.2 (Pin_2)
- new net: J200.3 (Pin_3), J6.TN, J70.3 (Pin_3)
- new net: J200.4 (Pin_4), J7.TN, J70.4 (Pin_4)
- new net: J200.5 (Pin_5), J70.5 (Pin_5), J8.TN
- new net: J200.10 (Pin_10), J70.6 (Pin_6), J9.TN
- new net Blue: J60.5 (Pin_5), J9.T
- new net Clock Out: J4.T, J50.6 (Pin_6)
- new net External Clock: J3.T, J50.4 (Pin_4)
- new net GND: J1.S, J2.S, J200.6 (Pin_6), J200.7 (Pin_7), J200.8 (Pin_8), J200.9 (Pin_9), J3.S, J4.S, J5.S, J6.S, J60.6 (Pin_6), J7.S, J8.S, J9.S
- new net Input: J1.T, J50.1 (Pin_1)
- new net Internal Clock: J3.TN, J50.5 (Pin_5)
- new net Pink: J60.3 (Pin_3), J7.T
- new net S&H: J2.TN, J50.3 (Pin_3)
- new net S&H Out: J5.T, J60.1 (Pin_1)
- new net Slew In: J2.T, J50.2 (Pin_2)
- new net Slew Out: J6.T, J60.2 (Pin_2)
- new net White: J1.TN, J60.4 (Pin_4), J8.T
