File: DMH_S_H_Noise_PCB_Conn/Power.kicad_sch (KiCad schematic)
At the start: 14 parts, among them J0 Conn_01x01, J100 IDC_02x08, J101 IDC_02x05

Commit message: Finished connectors PCB
Parts:
- removed C1, C2: 47uF, Capacitor_THT:CP_Radial_D5.0mm_P2.00mm, symbol Device:C_Polarized
- removed C3: 47uF, Capacitor_THT:CP_Radial_D4.0mm_P1.50mm, symbol Device:C_Polarized
- removed C4, C5, C6: 100nF, Capacitor_THT:C_Disc_D4.3mm_W1.9mm_P5.00mm, symbol Device:C
- removed D1, D3, D5: SB140+, Diode_THT:D_DO-41_SOD81_P10.16mm_Horizontal, symbol SynthStuff:Power_Bus_Schotty_+
- removed D2, D4: SB140-, Diode_THT:D_DO-41_SOD81_P10.16mm_Horizontal, symbol SynthStuff:Power_Bus_Schotty_-
- removed J0: Conn_01x01, Connector_PinHeader_2.54mm:PinHeader_1x01_P2.54mm_Vertical, symbol Connector_Generic:Conn_01x01
- removed J100: IDC_02x08, SynthStuff:IDC-Header_2x08_P2.54mm_Vertical_Eurorack, symbol SynthStuff:Eurorack_Power_Connector_16Pin
- removed J101: IDC_02x05, SynthStuff:IDC-Header_2x05_P2.54mm_Vertical_Eurorack, symbol SynthStuff:Eurorack_Power_Connector_10Pin
Other:
- note removed: "Delete what's not needed!"
