File: DMH_S_H_Noise_PCB_Conn/DMH_S_H_Noise_PCB_Conn.kicad_pcb (KiCad board)
At the start: 2 copper layers, 48 x 175 mm, 0 parts

Commit message: Finished connectors PCB
Parts:
- added J1: TS_Jack_6.35mm_Sw, SynthStuff:CUI_MJ-63052A, F.Cu at (58.5, 171.8)
- added J2: TS_Jack_6.35mm_Sw, SynthStuff:CUI_MJ-63052A, F.Cu at (58.5, 190.2)
- added J3: TS_Jack_6.35mm_Sw, SynthStuff:CUI_MJ-63052A, F.Cu at (75.0, 171.8)
- added J4: TS_Jack_6.35mm_Sw, SynthStuff:CUI_MJ-63052A, F.Cu at (75.0, 190.2)
- added J5: TS_Jack_6.35mm_Sw, SynthStuff:CUI_MJ-63052A, F.Cu at (91.5, 171.8)
- added J50: Conn_01x06, Connector_PinHeader_2.54mm:PinHeader_1x06_P2.54mm_Vertical, F.Cu at (52.4, 161.1)
- added J6: TS_Jack_6.35mm_Sw, SynthStuff:CUI_MJ-63052A, F.Cu at (91.5, 190.2)
- added J60: Conn_01x06, Connector_PinHeader_2.54mm:PinHeader_1x06_P2.54mm_Vertical, F.Cu at (81.3, 161.1)
- added J7: TS_Jack_6.35mm_Sw, SynthStuff:CUI_MJ-63052A, F.Cu at (58.5, 208.8)
- added J70: Conn_01x06, Connector_PinHeader_2.54mm:PinHeader_1x06_P2.54mm_Vertical, F.Cu at (97.7, 161.1)
- added J8: TS_Jack_6.35mm_Sw, SynthStuff:CUI_MJ-63052A, F.Cu at (75.0, 208.8)
- added J9: TS_Jack_6.35mm_Sw, SynthStuff:CUI_MJ-63052A, F.Cu at (91.5, 208.8)
Routing:
- net Net-(J70-Pin_1): track 0.00 -> 73.7 mm
- net Net-(J70-Pin_4): track 0.00 -> 73.2 mm
- net /Inputs and Outputs/Pink: track 0.00 -> 66.4 mm
- net Net-(J70-Pin_6): track 0.00 -> 62.2 mm
- net Net-(J70-Pin_5): track 0.00 -> 60.4 mm
- net /Inputs and Outputs/White: track 0.00 -> 53.2 mm
- net /Inputs and Outputs/Blue: track 0.00 -> 49.4 mm
- net /Inputs and Outputs/Slew In: track 0.00 -> 38.9 mm
- net Net-(J70-Pin_3): track 0.00 -> 36.7 mm
- net /Inputs and Outputs/Clock Out: track 0.00 -> 36.3 mm
- net /Inputs and Outputs/S&H: track 0.00 -> 34.8 mm
- net /Inputs and Outputs/Slew Out: track 0.00 -> 27.7 mm
- net /Inputs and Outputs/Internal Clock: track 0.00 -> 21.3 mm
- net /Inputs and Outputs/Input: track 0.00 -> 19.9 mm
- net /Inputs and Outputs/External Clock: track 0.00 -> 14.7 mm
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- added copper zone on B.Cu, net GND
- added copper zone on F.Cu, net GND
Other:
- board size 48 x 175 mm -> 48 x 58.5 mm

Commit message: Generated Gerbers
Other:
- board text added: "Mk1.0 - December 2024"
- board text removed: "Mk1.0 - Month Year"
Changed lines of the file:
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@@
 			(plot_on_all_layers_selection 0x0000000_00000000)
 			(disableapertmacros no)
-			(usegerberextensions no)
+			(usegerberextensions yes)
 			(usegerberattributes yes)
 			(usegerberadvancedattributes yes)
@@
 			(plotinvisibletext no)
 			(sketchpadsonfab no)
-			(subtractmaskfromsilk no)
+			(subtractmaskfromsilk yes)
 			(outputformat 1)
 			(mirror no)
-			(drillshape 1)
+			(drillshape 0)
 			(scaleselection 1)
-			(outputdirectory "")
+			(outputdirectory "Gerbers/")
 		)
 	)
@@
 		(at 75 171.75 180)
 		(property "Reference" "J3"
-			(at -4.075 -7 360)
+			(at -4.075 -7 0)
 			(layer "F.SilkS")
 			(effects
@@
 		)
 		(property "Value" "TS_Jack_6.35mm_Sw"
-			(at 1.005 9.035 360)
+			(at 1.005 9.035 0)
 			(layer "F.Fab")
 			(effects
@@
 		(at 75 208.75 180)
 		(property "Reference" "J8"
-			(at -4.075 -7 360)
+			(at -4.075 -7 0)
 			(layer "F.SilkS")
 			(effects
@@
 		)
 		(property "Value" "TS_Jack_6.35mm_Sw"
-			(at 1.005 9.035 360)
+			(at 1.005 9.035 0)
 			(layer "F.Fab")
 			(effects
@@
 		)
 		(property "Function" "White"
-			(at 0 0 360)
+			(at 0 0 0)
 			(layer "B.SilkS")
 			(effects
@@
 		(tags "Through hole pin header THT 1x06 2.54mm single row")
 		(property "Reference" "J70"
-			(at 2.4 6.4 -180)
+			(at 2.4 6.4 180)
 			(layer "B.SilkS")
 			(effects
@@
 		)
 		(fp_text user "${REFERENCE}"
-			(at 0 6.35 360)
+			(at 0 6.35 0)
 			(layer "F.Fab")
 			(effects
@@
 		(at 75 190.25 180)
 		(property "Reference" "J4"
-			(at -4.075 -7 360)
+			(at -4.075 -7 0)
 			(layer "F.SilkS")
 			(effects
@@
 		)
 		(property "Value" "TS_Jack_6.35mm_Sw"
-			(at 1.005 9.035 360)
+			(at 1.005 9.035 0)
 			(layer "F.Fab")
 			(effects
@@
 		)
 		(property "Function" "Clock Out"
-			(at 0 0 360)
+			(at 0 0 0)
 			(layer "B.SilkS")
 			(effects
@@
 		(tags "Through hole pin header THT 1x06 2.54mm single row")
 		(property "Reference" "J50"
-			(at -2.4 6.4 -180)
+			(at -2.4 6.4 180)
 			(layer "B.SilkS")
 			(effects
@@
 		)
 		(fp_text user "${REFERENCE}"
-			(at 0 6.35 360)
+			(at 0 6.35 0)
 			(layer "F.Fab")
 			(effects
@@
 		(tags "Through hole pin header THT 1x06 2.54mm single row")
 		(property "Reference" "J60"
-			(at 2.4 6.35 -180)
+			(at 2.4 6.35 180)
 			(layer "B.SilkS")
 			(effects
@@
 		)
 		(fp_text user "${REFERENCE}"
-			(at 0 6.35 360)
+			(at 0 6.35 0)
 			(layer "F.Fab")
 			(effects
@@
 		(layer "User.9")
 	)
-	(gr_text "Mk1.0 - Month Year"
+	(gr_text "Mk1.0 - December 2024"
 		(at 98 199.75 90)
 		(layer "B.SilkS")
