File: DMH_S_H_Noise_PANEL/DMH_S_H_Noise_PANEL.kicad_pcb (KiCad board)
At the start: 2 copper layers, 50 x 200 mm, 20 parts, among them J0 Panel_GND_Solder_Wire_Pad

Commit message: Generated Gerbers
Other:
- board text added: "548"
- board text added: "Mk1.0 - December 2024"
- board text removed: "Mk1.0 - Month Year"
- board text removed: "mki"
Changed lines of the file:
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@@
 			(plot_on_all_layers_selection 0x0000000_00000000)
 			(disableapertmacros no)
-			(usegerberextensions no)
+			(usegerberextensions yes)
 			(usegerberattributes yes)
 			(usegerberadvancedattributes yes)
@@
 			(plotinvisibletext no)
 			(sketchpadsonfab no)
-			(subtractmaskfromsilk no)
+			(subtractmaskfromsilk yes)
 			(outputformat 1)
 			(mirror no)
-			(drillshape 1)
+			(drillshape 0)
 			(scaleselection 1)
-			(outputdirectory "")
+			(outputdirectory "Gerbers/")
 		)
 	)
@@
 		(layer "F.Cu")
 		(at 75 71)
+		(descr "Based on Alpha RD901F-40-DD0")
 		(property "Reference" "H5"
 			(at 0 -7.9 0)
@@
 		(layer "F.Cu")
 		(at 87.5 108.25)
+		(descr "Based on Alpha RD901F-40-DD0")
 		(property "Reference" "H7"
 			(at 0 -7.9 0)
@@
 		(layer "F.Cu")
 		(at 62.5 108.25)
+		(descr "Based on Alpha RD901F-40-DD0")
 		(property "Reference" "H6"
 			(at 0 -7.9 0)
@@
 		(layer "User.9")
 	)
-	(gr_text "Mk1.0 - Month Year"
+	(gr_text "Mk1.0 - December 2024"
 		(at 75 222.95 0)
 		(layer "B.SilkS")
@@
 		)
 	)
-	(gr_text "mki"
+	(gr_text "548"
 		(at 75 225.75 0)
 		(layer "F.SilkS")
@@
 			)
 		)
-		(render_cache "mki" 0
+		(render_cache "548" 0
 			(polygon
 				(pts
-					(xy 72.167027 227.257211) (xy 72.338999 227.239499) (xy 72.513879 227.175197) (xy 72.655781 227.060611)
-					(xy 72.725244 226.954594) (xy 73.729693 224.876454) (xy 73.793806 224.837985) (xy 73.871598 224.926035)
-					(xy 73.871598 227.202501) (xy 74.724738 227.202501) (xy 74.724738 224.773017) (xy 74.713034 224.577881)
-					(xy 74.678711 224.409973) (xy 74.611659 224.244885) (xy 74.501713 224.091577) (xy 74.416137 224.0122)
-					(xy 74.264106 223.913135) (xy 74.104121 223.84861) (xy 73.923735 223.814286) (xy 73.837404 223.810456)
-					(xy 73.652416 223.828295) (xy 73.461285 223.893864) (xy 73.299919 224.002658) (xy 73.164191 224.149438)
-					(xy 73.067695 224.296991) (xy 72.999651 224.429367) (xy 72.249947 226.059566) (xy 72.167027 226.122825)
-					(xy 72.083252 226.059566) (xy 71.333548 224.429367) (xy 71.247286 224.265807) (xy 71.147992 224.122559)
-					(xy 71.008278 223.981746) (xy 70.842237 223.879792) (xy 70.645745 223.821938) (xy 70.495795 223.810456)
-					(xy 70.306819 223.829233) (xy 70.137584 223.881153) (xy 69.974502 223.969662) (xy 69.917062 224.0122)
-					(xy 69.786256 224.145023) (xy 69.689351 224.311825) (xy 69.634573 224.490692) (xy 69.611412 224.671876)
-					(xy 69.608461 224.773017) (xy 69.608461 227.202501) (xy 70.461601 227.202501) (xy 70.461601 224.930309)
-					(xy 70.539393 224.84226) (xy 70.603506 224.880728) (xy 71.607955 226.967417) (xy 71.720221 227.109366)
-					(xy 71.874784 227.203123) (xy 72.057949 227.2504)
+					(xy 69.027163 226.355344) (xy 69.027163 227.202501) (xy 71.69344 227.202501) (xy 71.880122 227.193377)
+					(xy 72.077528 227.159535) (xy 72.247627 227.102731) (xy 72.413998 227.010279) (xy 72.548586 226.892855)
+					(xy 72.565387 226.874238) (xy 72.67299 226.716619) (xy 72.740282 226.556729) (xy 72.779885 226.381893)
+					(xy 72.791067 226.219423) (xy 72.778225 226.048247) (xy 72.731552 225.86063) (xy 72.652029 225.689917)
+					(xy 72.540998 225.540189) (xy 72.443144 225.448348) (xy 72.282812 225.345833) (xy 72.10957 225.279551)
+					(xy 71.928871 225.242904) (xy 71.748855 225.228762) (xy 71.683182 225.227797) (xy 70.1 225.227797)
+					(xy 70.031612 225.149151) (xy 70.061532 224.805501) (xy 70.12479 224.743097) (xy 72.667969 224.743097)
+					(xy 72.667969 223.865166) (xy 69.507589 223.865166) (xy 69.337578 223.896764) (xy 69.209599 224.016887)
+					(xy 69.169068 224.184025) (xy 69.095551 225.52614) (xy 69.128585 225.704242) (xy 69.265893 225.816214)
+					(xy 69.394749 225.834741) (xy 71.590003 225.834741) (xy 71.759045 225.863583) (xy 71.825087 225.908258)
+					(xy 71.89368 226.071414) (xy 71.89433 226.092905) (xy 71.840825 226.260292) (xy 71.825087 226.277553)
+					(xy 71.667487 226.350041) (xy 71.590003 226.355344)
 				)
 			)
 			(polygon
 				(pts
-					(xy 75.201744 223.865166) (xy 75.201744 227.202501) (xy 76.098482 227.202501) (xy 76.098482 225.727029)
-					(xy 77.685938 227.06487) (xy 77.814133 227.181985) (xy 77.832973 227.202501) (xy 79.15628 227.202501)
-					(xy 79.033072 227.083091) (xy 79.028908 227.079402) (xy 77.073866 225.485107) (xy 77.044801 225.430397)
-					(xy 77.073866 225.376541) (xy 78.896406 223.954071) (xy 78.98531 223.865166) (xy 77.744923 223.865166)
-					(xy 77.621966 223.992208) (xy 77.608147 224.003652) (xy 76.098482 225.232926) (xy 76.098482 223.865166)
+					(xy 76.336053 223.825618) (xy 76.507744 223.881624) (xy 76.659264 223.9857) (xy 76.709483 224.040683)
+					(xy 76.797322 224.201977) (xy 76.839925 224.384585) (xy 76.85075 224.564434) (xy 76.85075 227.202501)
+					(xy 75.958287 227.202501) (xy 75.958287 226.718655) (xy 73.650192 226.718655) (xy 73.478487 226.707155)
+					(xy 73.299071 226.656583) (xy 73.155234 226.55196) (xy 73.133058 226.524868) (xy 73.055928 226.365762)
+					(xy 73.03299 226.189503) (xy 73.055109 226.03937) (xy 73.132881 225.891161) (xy 74.390492 225.891161)
+					(xy 74.444347 225.944161) (xy 75.958287 225.944161) (xy 75.958287 224.9286) (xy 75.884769 224.832002)
+					(xy 75.806978 224.861066) (xy 74.424686 225.837305) (xy 74.390492 225.891161) (xy 73.132881 225.891161)
+					(xy 73.135572 225.886032) (xy 73.216676 225.797661) (xy 73.356123 225.686852) (xy 75.713799 223.976297)
+					(xy 75.833278 223.899173) (xy 76.001351 223.830922) (xy 76.174564 223.810456)
 				)
 			)
 			(polygon
 				(pts
-					(xy 79.474284 223.865166) (xy 79.474284 227.202501) (xy 80.365893 227.202501) (xy 80.365893 223.865166)
+					(xy 80.068782 223.873072) (xy 80.243466 223.903166) (xy 80.426777 223.966089) (xy 80.587462 224.05825)
+					(xy 80.72493 224.178896) (xy 80.839011 224.32981) (xy 80.91441 224.487485) (xy 80.960908 224.667641)
+					(xy 80.974546 224.843969) (xy 80.973169 224.89778) (xy 80.947008 225.076806) (xy 80.888634 225.238483)
+					(xy 80.784128 225.397191) (xy 80.641155 225.52272) (xy 80.747146 225.5939) (xy 80.865277 225.727684)
+					(xy 80.948158 225.893129) (xy 80.995842 226.081216) (xy 81.00874 226.253617) (xy 81.002422 226.36368)
+					(xy 80.961044 226.551527) (xy 80.884977 226.722969) (xy 80.778786 226.874238) (xy 80.653549 226.994955)
+					(xy 80.501069 227.091181) (xy 80.31791 227.159535) (xy 80.133894 227.193377) (xy 79.959839 227.202501)
+					(xy 78.289462 227.202501) (xy 78.115408 227.193377) (xy 77.931391 227.159535) (xy 77.748232 227.091181)
+					(xy 77.595753 226.994955) (xy 77.470516 226.874238) (xy 77.3966 226.775819) (xy 77.309984 226.610683)
+					(xy 77.256537 226.427886) (xy 77.240562 226.253617) (xy 77.246293 226.137852) (xy 77.252227 226.107438)
+					(xy 78.171493 226.107438) (xy 78.173286 226.140245) (xy 78.239881 226.298924) (xy 78.33093 226.368)
+					(xy 78.499756 226.398942) (xy 79.749546 226.398942) (xy 79.858547 226.387797) (xy 80.009421 226.298924)
+					(xy 80.028457 226.272202) (xy 80.077809 226.107438) (xy 80.076473 226.08141) (xy 80.004291 225.921935)
+					(xy 79.921109 225.857787) (xy 79.749546 225.826192) (xy 78.499756 225.826192) (xy 78.402069 225.8343)
+					(xy 78.24501 225.921935) (xy 78.229089 225.941512) (xy 78.171493 226.107438) (xy 77.252227 226.107438)
+					(xy 77.283931 225.944953) (xy 77.35675 225.772118) (xy 77.464804 225.628367) (xy 77.608147 225.52272)
+					(xy 77.568902 225.494755) (xy 77.435365 225.360405) (xy 77.340778 225.194279) (xy 77.291476 225.027262)
+					(xy 77.285673 224.963648) (xy 78.191155 224.963648) (xy 78.250139 225.128634) (xy 78.323404 225.1942)
+					(xy 78.494626 225.232926) (xy 79.754675 225.232926) (xy 79.855734 225.221823) (xy 79.999162 225.128634)
+					(xy 80.058147 224.963648) (xy 79.999162 224.798662) (xy 79.925898 224.736843) (xy 79.754675 224.698645)
+					(xy 78.494626 224.698645) (xy 78.402514 224.707723) (xy 78.250139 224.798662) (xy 78.191155 224.963648)
+					(xy 77.285673 224.963648) (xy 77.274756 224.843969) (xy 77.288394 224.667641) (xy 77.334891 224.487485)
+					(xy 77.41029 224.32981) (xy 77.524372 224.178896) (xy 77.640766 224.073758) (xy 77.798171 223.977482)
+					(xy 77.978285 223.910336) (xy 78.150297 223.876538) (xy 78.338189 223.865166) (xy 79.911113 223.865166)
 				)
 			)
