File: DMH_S_H_Noise_PCB/DMH_S_H_Noise_PCB.kicad_pcb (KiCad board)
At the start: 2 copper layers, 48 x 120.5 mm, 82 parts, among them J0 Conn_01x01, J100 IDC_02x05, J200 IDC_02x05, J50 Conn_01x06, J60 Conn_01x06, J70 Conn_01x06, Q1 BC548, Q2 J113, Q3 BC548, SW1 SW_Push, SW2 SW_SPDT_321, U1 TL074, U2 TL074, U3 TL074

Commit message: Finished connectors PCB
Parts:
- J50, J60, J70: footprint Connector_PinHeader_2.54mm:PinHeader_1x06_P2.54mm_Vertical -> Connector_PinSocket_2.54mm:PinSocket_1x06_P2.54mm_Vertical
Changed lines of the file:
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@@
 		)
 	)
-	(footprint "Connector_PinHeader_2.54mm:PinHeader_1x06_P2.54mm_Vertical"
+	(footprint "Connector_PinSocket_2.54mm:PinSocket_1x06_P2.54mm_Vertical"
 		(locked yes)
 		(layer "B.Cu")
 		(at 52.35 161.1 -90)
-		(descr "Through hole straight pin header, 1x06, 2.54mm pitch, single row")
-		(tags "Through hole pin header THT 1x06 2.54mm single row")
+		(descr "Through hole straight socket strip, 1x06, 2.54mm pitch, single row (from Kicad 4.0.7), script generated")
+		(tags "Through hole socket strip THT 1x06 2.54mm single row")
 		(property "Reference" "J50"
-			(at -3 -1.75 0)
+			(at -2.1 -2.4 180)
 			(layer "B.SilkS")
-			(hide yes)
 			(effects
 				(font
@@
 		)
 		(property "Value" "Conn_01x06"
-			(at 0 -15.03 90)
+			(at 0 -15.47 90)
 			(layer "B.Fab")
+			(hide yes)
 			(effects
 				(font
@@
 			)
 		)
-		(property "Footprint" "Connector_PinHeader_2.54mm:PinHeader_1x06_P2.54mm_Vertical"
+		(property "Footprint" "Connector_PinSocket_2.54mm:PinSocket_1x06_P2.54mm_Vertical"
 			(at 0 0 90)
 			(unlocked yes)
@@
 		)
 		(property "Function" ""
-			(at 0 0 90)
+			(at 0 0 -90)
 			(unlocked yes)
 			(layer "B.Fab")
@@
 		(attr through_hole)
 		(fp_line
-			(start -1.33 1.33)
-			(end -1.33 0)
+			(start 1.33 1.33)
+			(end 0 1.33)
 			(stroke
 				(width 0.12)
@@
 		)
 		(fp_line
-			(start 0 1.33)
-			(end -1.33 1.33)
+			(start 1.33 0)
+			(end 1.33 1.33)
 			(stroke
 				(width 0.12)
@@
 		(fp_line
 			(start -1.8 1.8)
-			(end 1.8 1.8)
+			(end -1.8 -14.45)
 			(stroke
 				(width 0.05)
@@
 		)
 		(fp_line
-			(start 1.8 1.8)
-			(end 1.8 -14.5)
+			(start 1.75 1.8)
+			(end -1.8 1.8)
 			(stroke
 				(width 0.05)
@@
 		)
 		(fp_line
-			(start -1.8 -14.5)
-			(end -1.8 1.8)
+			(start -1.8 -14.45)
+			(end 1.75 -14.45)
 			(stroke
 				(width 0.05)
@@
 		)
 		(fp_line
-			(start 1.8 -14.5)
-			(end -1.8 -14.5)
+			(start 1.75 -14.45)
+			(end 1.75 1.8)
 			(stroke
 				(width 0.05)
@@
 		)
 		(fp_line
-			(start -0.635 1.27)
-			(end -1.27 0.635)
+			(start -1.27 1.27)
+			(end -1.27 -13.97)
 			(stroke
 				(width 0.1)
@@
 		)
 		(fp_line
-			(start 1.27 1.27)
-			(end -0.635 1.27)
+			(start 0.635 1.27)
+			(end -1.27 1.27)
 			(stroke
 				(width 0.1)
@@
 		)
 		(fp_line
-			(start -1.27 0.635)
-			(end -1.27 -13.97)
+			(start 1.27 0.635)
+			(end 0.635 1.27)
 			(stroke
 				(width 0.1)
@@
 		(fp_line
 			(start 1.27 -13.97)
-			(end 1.27 1.27)
+			(end 1.27 0.635)
 			(stroke
 				(width 0.1)
@@
 		)
 		(fp_text user "${REFERENCE}"
-			(at 0 -6.35 0)
+			(at 0 -6.35 180)
 			(layer "B.Fab")
 			(effects
@@
 			(pintype "passive")
 		)
-		(model "${KICAD8_3DMODEL_DIR}/Connector_PinHeader_2.54mm.3dshapes/PinHeader_1x06_P2.54mm_Vertical.wrl"
+		(model "${KICAD8_3DMODEL_DIR}/Connector_PinSocket_2.54mm.3dshapes/PinSocket_1x06_P2.54mm_Vertical.wrl"
 			(offset
 				(xyz 0 0 0)
@@
 		)
 	)
-	(footprint "Connector_PinHeader_2.54mm:PinHeader_1x06_P2.54mm_Vertical"
+	(footprint "Connector_PinSocket_2.54mm:PinSocket_1x06_P2.54mm_Vertical"
 		(locked yes)
 		(layer "B.Cu")
 		(at 81.35 161.1 90)
-		(descr "Through hole straight pin header, 1x06, 2.54mm pitch, single row")
-		(tags "Through hole pin header THT 1x06 2.54mm single row")
+		(descr "Through hole straight socket strip, 1x06, 2.54mm pitch, single row (from Kicad 4.0.7), script generated")
+		(tags "Through hole socket strip THT 1x06 2.54mm single row")
 		(property "Reference" "J60"
-			(at -2.25 -6.35 0)
+			(at 2.1 -13.1 0)
 			(layer "B.SilkS")
-			(hide yes)
 			(effects
 				(font
@@
 		)
 		(property "Value" "Conn_01x06"
-			(at 0 -15.03 90)
+			(at 0 -15.47 -90)
 			(layer "B.Fab")
+			(hide yes)
 			(effects
 				(font
@@
 			)
 		)
-		(property "Footprint" "Connector_PinHeader_2.54mm:PinHeader_1x06_P2.54mm_Vertical"
+		(property "Footprint" "Connector_PinSocket_2.54mm:PinSocket_1x06_P2.54mm_Vertical"
 			(at 0 0 -90)
 			(unlocked yes)
@@
 		)
 		(property "Function" ""
-			(at 0 0 -90)
+			(at 0 0 90)
 			(unlocked yes)
 			(layer "B.Fab")
@@
 		)
 		(fp_line
-			(start 0 1.33)
-			(end -1.33 1.33)
+			(start 1.33 0)
+			(end 1.33 1.33)
 			(stroke
 				(width 0.12)
@@
 		)
 		(fp_line
-			(start -1.33 1.33)
-			(end -1.33 0)
+			(start 1.33 1.33)
+			(end 0 1.33)
 			(stroke
 				(width 0.12)
@@
 		)
 		(fp_line
-			(start 1.8 -14.5)
-			(end -1.8 -14.5)
+			(start 1.75 -14.45)
+			(end 1.75 1.8)
 			(stroke
 				(width 0.05)
@@
 		)
 		(fp_line
-			(start -1.8 -14.5)
-			(end -1.8 1.8)
+			(start -1.8 -14.45)
+			(end 1.75 -14.45)
 			(stroke
 				(width 0.05)
@@
 		)
 		(fp_line
-			(start 1.8 1.8)
-			(end 1.8 -14.5)
+			(start 1.75 1.8)
+			(end -1.8 1.8)
 			(stroke
 				(width 0.05)
@@
 		(fp_line
 			(start -1.8 1.8)
-			(end 1.8 1.8)
+			(end -1.8 -14.45)
 			(stroke
 				(width 0.05)
@@
 		(fp_line
 			(start 1.27 -13.97)
-			(end 1.27 1.27)
+			(end 1.27 0.635)
 			(stroke
 				(width 0.1)
@@
 		)
 		(fp_line
-			(start -1.27 0.635)
-			(end -1.27 -13.97)
+			(start 1.27 0.635)
+			(end 0.635 1.27)
 			(stroke
 				(width 0.1)
@@
 		)
 		(fp_line
-			(start 1.27 1.27)
-			(end -0.635 1.27)
+			(start 0.635 1.27)
+			(end -1.27 1.27)
 			(stroke
 				(width 0.1)
@@
 		)
 		(fp_line
-			(start -0.635 1.27)
-			(end -1.27 0.635)
+			(start -1.27 1.27)
+			(end -1.27 -13.97)
 			(stroke
 				(width 0.1)
@@
 			(pintype "passive")
 		)
-		(model "${KICAD8_3DMODEL_DIR}/Connector_PinHeader_2.54mm.3dshapes/PinHeader_1x06_P2.54mm_Vertical.wrl"
+		(model "${KICAD8_3DMODEL_DIR}/Connector_PinSocket_2.54mm.3dshapes/PinSocket_1x06_P2.54mm_Vertical.wrl"
 			(offset
 				(xyz 0 0 0)
@@
 		)
 	)
-	(footprint "Connector_PinHeader_2.54mm:PinHeader_1x06_P2.54mm_Vertical"
+	(footprint "Connector_PinSocket_2.54mm:PinSocket_1x06_P2.54mm_Vertical"
 		(locked yes)
 		(layer "B.Cu")
 		(at 97.65 161.1 90)
-		(descr "Through hole straight pin header, 1x06, 2.54mm pitch, single row")
-		(tags "Through hole pin header THT 1x06 2.54mm single row")
+		(descr "Through hole straight socket strip, 1x06, 2.54mm pitch, single row (from Kicad 4.0.7), script generated")
+		(tags "Through hole socket strip THT 1x06 2.54mm single row")
 		(property "Reference" "J70"
-			(at -2.25 -6.37 0)
+			(at 2.1 -12.9 0)
 			(layer "B.SilkS")
-			(hide yes)
 			(effects
 				(font
@@
 		)
 		(property "Value" "Conn_01x06"
-			(at 0 -15.03 90)
+			(at 0 -15.47 -90)
 			(layer "B.Fab")
+			(hide yes)
 			(effects
 				(font
@@
 			)
 		)
-		(property "Footprint" "Connector_PinHeader_2.54mm:PinHeader_1x06_P2.54mm_Vertical"
+		(property "Footprint" "Connector_PinSocket_2.54mm:PinSocket_1x06_P2.54mm_Vertical"
 			(at 0 0 -90)
 			(unlocked yes)
@@
 		)
 		(property "Function" ""
-			(at 0 0 -90)
+			(at 0 0 90)
 			(unlocked yes)
 			(layer "B.Fab")
@@
 		)
 		(fp_line
-			(start 0 1.33)
-			(end -1.33 1.33)
+			(start 1.33 0)
+			(end 1.33 1.33)
 			(stroke
 				(width 0.12)
@@
 		)
 		(fp_line
-			(start -1.33 1.33)
-			(end -1.33 0)
+			(start 1.33 1.33)
+			(end 0 1.33)
 			(stroke
 				(width 0.12)
@@
 		)
 		(fp_line
-			(start 1.8 -14.5)
-			(end -1.8 -14.5)
+			(start 1.75 -14.45)
+			(end 1.75 1.8)
 			(stroke
 				(width 0.05)
@@
 		)
 		(fp_line
-			(start -1.8 -14.5)
-			(end -1.8 1.8)
+			(start -1.8 -14.45)
+			(end 1.75 -14.45)
 			(stroke
 				(width 0.05)
@@
 		)
 		(fp_line
-			(start 1.8 1.8)
-			(end 1.8 -14.5)
+			(start 1.75 1.8)
+			(end -1.8 1.8)
 			(stroke
 				(width 0.05)
@@
 		(fp_line
 			(start -1.8 1.8)
-			(end 1.8 1.8)
+			(end -1.8 -14.45)
 			(stroke
 				(width 0.05)
@@
 		(fp_line
 			(start 1.27 -13.97)
-			(end 1.27 1.27)
+			(end 1.27 0.635)
 			(stroke
 				(width 0.1)
@@
 		)
 		(fp_line
-			(start -1.27 0.635)
-			(end -1.27 -13.97)
+			(start 1.27 0.635)
+			(end 0.635 1.27)
 			(stroke
 				(width 0.1)
@@
 		)
 		(fp_line
-			(start 1.27 1.27)
-			(end -0.635 1.27)
+			(start 0.635 1.27)
+			(end -1.27 1.27)
 			(stroke
 				(width 0.1)
@@
 		)
 		(fp_line
-			(start -0.635 1.27)
-			(end -1.27 0.635)
+			(start -1.27 1.27)
+			(end -1.27 -13.97)
 			(stroke
 				(width 0.1)
@@
 			(pintype "passive")
 		)
-		(model "${KICAD8_3DMODEL_DIR}/Connector_PinHeader_2.54mm.3dshapes/PinHeader_1x06_P2.54mm_Vertical.wrl"
+		(model "${KICAD8_3DMODEL_DIR}/Connector_PinSocket_2.54mm.3dshapes/PinSocket_1x06_P2.54mm_Vertical.wrl"
 			(offset
 				(xyz 0 0 0)

Commit message: Generated Gerbers
Other:
- board text added: "Mk1.0 - December 2024"
- board text removed: "Mk1.0 - Month Year"
Changed lines of the file:
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@@
 			(plot_on_all_layers_selection 0x0000000_00000000)
 			(disableapertmacros no)
-			(usegerberextensions no)
+			(usegerberextensions yes)
 			(usegerberattributes yes)
 			(usegerberadvancedattributes yes)
@@
 			(plotinvisibletext no)
 			(sketchpadsonfab no)
-			(subtractmaskfromsilk no)
+			(subtractmaskfromsilk yes)
 			(outputformat 1)
 			(mirror no)
-			(drillshape 1)
+			(drillshape 0)
 			(scaleselection 1)
-			(outputdirectory "")
+			(outputdirectory "Gerbers/")
 		)
 	)
@@
 		(tags "Through hole socket strip THT 1x06 2.54mm single row")
 		(property "Reference" "J50"
-			(at -2.1 -2.4 180)
+			(at -2.1 -0.15 180)
 			(layer "B.SilkS")
 			(effects
@@
 		)
 		(property "Value" "100nF"
-			(at 2.5 0 90)
+			(at 2.95 0 90)
 			(layer "B.SilkS")
 			(effects
@@
 	)
 	(gr_rect
-		(start 53.6 146.5)
-		(end 55.6 156.5)
+		(start 53.6 142.75)
+		(end 55.6 152.75)
 		(stroke
 			(width 0.1)
@@
 		(layer "User.9")
 	)
-	(gr_text "Mk1.0 - Month Year"
-		(at 52.1 151.25 -90)
+	(gr_text "Mk1.0 - December 2024"
+		(at 52.1 147.5 270)
 		(layer "B.SilkS")
 		(effects
